Commit message: Changed the urdf files to match the deepracer specifications (#12)
* changed the urdf files to match the deepracer specifications

* fixing the -0 typo in racecar xacro

* reverting from RGB to BGR

File: simulation_ws/src/deepracer_simulation/urdf/macros.xacro (robot description, xacro)
@@ -4,5 +4,5 @@
 <xacro:macro name="chassis_inertial_params">
   <origin xyz="0.1477 0 0" rpy="0 0 0" />
-  <mass value="4.0" />
+  <mass value="5.0" />
   <inertia ixx="0.010609" ixy="0"          ixz="0"
                           iyy="0.050409"   iyz="0"
@@ -10,5 +10,5 @@
 </xacro:macro>
 <xacro:macro name="left_wheels_inertial_params">
-  <origin xyz="0 0 -0.0225" rpy="0 0 0" />
+  <origin xyz="0 0 -0.0125" rpy="0 0 0" />
   <mass value="0.34055" />
   <inertia ixx="0.00026046" ixy="0"          ixz="0"
@@ -17,5 +17,5 @@
 </xacro:macro>
 <xacro:macro name="right_wheels_inertial_params">
-  <origin xyz="0 0 0.0225" rpy="0 0 0" />
+  <origin xyz="0 0 0.0125" rpy="0 0 0" />
   <mass value="0.34055" />
   <inertia ixx="0.00026046" ixy="0"          ixz="0"
@@ -40,5 +40,5 @@
   <origin xyz="0 0 0" rpy="0 0 0" />
   <geometry>
-    <mesh filename="package://deepracer_simulation/meshes/left_rear_wheel.STL" />
+    <mesh scale="0.6 0.6 0.6" filename="package://deepracer_simulation/meshes/left_rear_wheel.STL" />
   </geometry>
 </xacro:macro>
@@ -46,5 +46,5 @@
   <origin xyz="0 0 0" rpy="0 0 0" />
   <geometry>
-    <mesh filename="package://deepracer_simulation/meshes/right_rear_wheel.STL" />
+    <mesh scale="0.6 0.6 0.6" filename="package://deepracer_simulation/meshes/right_rear_wheel.STL" />
   </geometry>
 </xacro:macro>
@@ -52,5 +52,5 @@
   <origin xyz="0 0 0" rpy="0 0 0" />
   <geometry>
-    <mesh filename="package://deepracer_simulation/meshes/left_front_wheel.STL" />
+    <mesh scale="0.6 0.6 0.6" filename="package://deepracer_simulation/meshes/left_front_wheel.STL" />
   </geometry>
 </xacro:macro>
@@ -58,5 +58,5 @@
   <origin xyz="0 0 0" rpy="0 0 0" />
   <geometry>
-    <mesh filename="package://deepracer_simulation/meshes/right_front_wheel.STL" />
+    <mesh scale="0.6 0.6 0.6" filename="package://deepracer_simulation/meshes/right_front_wheel.STL" />
   </geometry>
 </xacro:macro>
@@ -64,5 +64,5 @@
   <origin xyz="0 0 0" rpy="0 0 0" />
   <geometry>
-    <mesh filename="package://deepracer_simulation/meshes/left_steering_hinge.STL" />
+    <mesh scale="0.6 0.6 0.6" filename="package://deepracer_simulation/meshes/left_steering_hinge.STL" />
   </geometry>
 </xacro:macro>
@@ -70,17 +70,17 @@
   <origin xyz="0 0 0" rpy="0 0 0" />
   <geometry>
-    <mesh filename="package://deepracer_simulation/meshes/right_steering_hinge.STL" />
+    <mesh scale="0.6 0.6 0.6" filename="package://deepracer_simulation/meshes/right_steering_hinge.STL" />
   </geometry>
 </xacro:macro>
 <xacro:macro name="left_wheels_collision_geometry">
-  <origin xyz="0 0 -0.0225" rpy="0 0 0" />
+  <origin xyz="0 0 -0.0125" rpy="0 0 0" />
   <geometry>
-    <cylinder length="0.045" radius="0.05" />
+    <cylinder length="0.025" radius="0.03" />
   </geometry>
 </xacro:macro>
 <xacro:macro name="right_wheels_collision_geometry">
-  <origin xyz="0 0 0.0225" rpy="0 0 0" />
+  <origin xyz="0 0 0.0125" rpy="0 0 0" />
   <geometry>
-    <cylinder length="0.045" radius="0.05" />
+    <cylinder length="0.025" radius="0.03" />
   </geometry>
 </xacro:macro>

File: simulation_ws/src/deepracer_simulation/urdf/racecar.xacro (robot description, xacro)
@@ -11,5 +11,5 @@
   </link>
   <joint name="base_link_joint" type="fixed">
-    <origin xyz="0 0 0.05" rpy="0 0 0" />
+    <origin xyz="0 0 0.03" rpy="0 0 0" />
     <parent link="base_link" />
     <child link="chassis" />
@@ -148,6 +148,6 @@
   <link name="zed_camera_link">
     <inertial>
-      <mass value="1e-5" />
-      <origin xyz="0 0 0" rpy="0 -0.26 0"/>
+      <mass value="1e-3" />
+      <origin xyz="0 0 0" rpy="0 0 0"/>
       <inertia ixx="1e-6" ixy="0" ixz="0" iyy="1e-6" iyz="0" izz="1e-6" />
     </inertial>
@@ -167,5 +167,5 @@
   </link>
   <joint name="zed_camera_joint" type="fixed">
-    <origin xyz="0.25 0 0.14" rpy="0 0 0"/>
+    <origin xyz="0.20 0 0.10" rpy="0 0.2731415 0"/>
     <parent link="chassis"/>
     <child link="zed_camera_link"/>
@@ -177,5 +177,5 @@
   <link name="camera_link"><!-- this needs to match the name in zed_wrapper/zed_tf.launch -->
     <inertial>
-      <mass value="1e-5" />
+      <mass value="1e-3" />
       <origin xyz="0 0 0" rpy="0 0 0"/>
       <inertia ixx="1e-6" ixy="0" ixz="0" iyy="1e-6" iyz="0" izz="1e-6" />
@@ -184,11 +184,11 @@
   <link name="zed_camera_right_link">
     <inertial>
-      <mass value="1e-5" />
-      <origin xyz="0 0 0" rpy="0 0 0"/>
+      <mass value="1e-3" />
+      <origin xyz="0 0.005 0" rpy="0 0 0"/>
       <inertia ixx="1e-6" ixy="0" ixz="0" iyy="1e-6" iyz="0" izz="1e-6" />
     </inertial>
   </link>
   <joint name="zed_camera_left_joint" type="fixed">
-    <origin xyz="0 0.06 0" rpy="0 0 0"/>
+    <origin xyz="0 0 0" rpy="0 0 0"/>
     <parent link="zed_camera_link"/>
     <child link="camera_link"/>
@@ -196,5 +196,5 @@
   </joint>
   <joint name="zed_camera_right_joint" type="fixed">
-    <origin xyz="0 -0.06 0" rpy="0 0 0"/>
+    <origin xyz="0 0 0" rpy="0 0 0"/>
     <parent link="zed_camera_link"/>
     <child link="zed_camera_right_link"/>
